Commit message: Clean up and update documents

File: urdf/sample.urdf (robot description, URDF)
Before this commit: robot robo, 13 links, 12 joints
Links:
- removed link root
- added link root_body, mass 1; collision cylinder length=0.5 radius=1; visual box size=0.2 0.2 0.4
Joints:
- joint l_elbow_pitch: limit lower=-2 upper=1.0 effort=0 velocity=1.0 -> lower=-2 upper=3.0 effort=0 velocity=1.0
- joint l_shoulder_pitch: limit lower=-1 upper=1.0 effort=0 velocity=1.0 -> lower=-3 upper=3.0 effort=0 velocity=1.0
- joint l_shoulder_roll: limit lower=-2 upper=1.0 effort=0 velocity=1.0 -> lower=-2 upper=3.0 effort=0 velocity=1.0
- joint l_shoulder_yaw: limit lower=-1 upper=1.0 effort=0 velocity=1.0 -> lower=-3 upper=3.0 effort=0 velocity=1.0
- joint l_wrist_pitch: limit lower=-2 upper=1.0 effort=0 velocity=1.0 -> lower=-2 upper=3.0 effort=0 velocity=1.0
- joint l_wrist_yaw: limit lower=-2 upper=1.0 effort=0 velocity=1.0 -> lower=-2 upper=3.0 effort=0 velocity=1.0
- joint r_elbow_pitch: limit lower=-2 upper=1.0 effort=0 velocity=1.0 -> lower=-2 upper=3.0 effort=0 velocity=1.0
- joint r_shoulder_pitch: limit lower=-1 upper=1.0 effort=0 velocity=1.0 -> lower=-3 upper=3.0 effort=0 velocity=1.0
- joint r_shoulder_roll: limit lower=-2 upper=1.0 effort=0 velocity=1.0 -> lower=-2 upper=3.0 effort=0 velocity=1.0
- joint r_shoulder_yaw: limit lower=-1 upper=1.0 effort=0 velocity=1.0 -> lower=-3 upper=3.0 effort=0 velocity=1.0
- joint r_wrist_pitch: limit lower=-2 upper=1.0 effort=0 velocity=1.0 -> lower=-2 upper=3.0 effort=0 velocity=1.0
